File: Hardware/VentilaTM/VentilaTM.kicad_pcb (KiCad board)
At the start: 2 copper layers, 70 x 100 mm, 64 parts, among them J1 PSU_IN, J10 endstop2, J11 FAN1, J12 FAN2, J13 Conn_01x06_Male, J2 M1Out, J3 M2Out, J4 BMP280, J5 BMP280_pacient, J6 Serial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

Commit message: update
fixed some issues, still W-I-P
Parts:
- removed G***: LOGO, logos:logo_Symme3D16x6_MUIELTHD
- added J14: 3v3spare, Connector_PinHeader_2.54mm:PinHeader_1x02_P2.54mm_Vertical, F.Cu at (24.8, 6.48)
- added J15: 3v3spare1, Connector_PinHeader_2.54mm:PinHeader_1x02_P2.54mm_Vertical, F.Cu at (28.4, 6.48)
- added J16: spare_pins, Connector_PinHeader_2.54mm:PinHeader_1x04_P2.54mm_Vertical, F.Cu at (19.8, 57.9)
- J13: moved to F.Cu
- moved C3 0.93 mm to (18.9, 83.4)
- moved J2 0.93 mm to (7.85, 81.8)
- moved C6 0.85 mm to (37.7, 71.0)
- turned J13 to 90 degrees
Connections:
- A1 pad 16: M_DIR -> M1_DIR
- A2 pad 16: M_DIR -> M2_DIR
- U2 pad 2: M_DIR -> M1_DIR
- U2 pad 21: CS1 -> Net-(J16-Pad4)
- U2 pad 22: ENDSTOP2 -> Net-(J16-Pad3)
- U2 pad 23: BTN2 -> Net-(J16-Pad2)
- U2 pad 24: (no net) -> CS1
- U2 pad 25: (no net) -> ENDSTOP2
- U2 pad 26: (no net) -> BTN2
- U2 pad 27: (no net) -> ENDSTOP1
- U2 pad 28: ENDSTOP1 -> Net-(J16-Pad1)
- U2 pad 8: (no net) -> M2_DIR
Routing:
- net M_DIR: track 50.1 -> 0.00 mm, vias 4 -> 0
- net M1_DIR: track 0.00 -> 33.5 mm, vias 0 -> 2
- net Net-(J16-Pad4): track 0.00 -> 28.0 mm
- net Net-(J16-Pad3): track 0.00 -> 23.0 mm
- net +3V3: track 323.9 -> 346.0 mm, vias 10 -> 14
- net M2_DIR: track 0.00 -> 21.2 mm, vias 0 -> 2
- net Net-(J16-Pad2): track 0.00 -> 18.3 mm
- net GND: track 115.3 -> 127.1 mm, vias 11 -> 15
- net Net-(J16-Pad1): track 0.00 -> 7.01 mm
- net CS1: track 30.5 -> 33.4 mm, vias 2 -> 0
- net +24V: track 167.0 -> 169.1 mm
- net ENDSTOP2: track 85.9 -> 84.4 mm
- net BTN2: track 88.5 -> 87.0 mm
- net Net-(A1-Pad4): track 8.13 -> 6.84 mm
- net Net-(A1-Pad3): track 8.03 -> 6.84 mm
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