File: Hardware/VentilaTM/VentilaTM.sch (KiCad schematic (older format))
At the start: 63 parts, among them J1 PSU_IN, J10 endstop2, J11 FAN1, J12 FAN2, J13 Conn_01x06_Male, J2 M1Out, J3 M2Out, J4 BMP280, J5 BMP280_pacient, J6 Serial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

Commit message: update
fixed some issues, still W-I-P
Parts:
- added J14: 3v3spare, Connector_PinHeader_2.54mm:PinHeader_1x02_P2.54mm_Vertical, symbol Connector:Conn_01x02_Male
- added J15: 3v3spare1, Connector_PinHeader_2.54mm:PinHeader_1x02_P2.54mm_Vertical, symbol Connector:Conn_01x02_Male
- added J16: spare_pins, Connector_PinHeader_2.54mm:PinHeader_1x04_P2.54mm_Vertical, symbol Connector:Conn_01x04_Male
Connections:
- net +3V3: now also J14.1 (Pin_1), J15.1 (Pin_1)
- net BTN2: now also U2.26 (GPA5); no longer U2.23 (GPA2)
- net CS1: now also U2.24 (GPA3); no longer U2.21 (GPA0)
- net ENDSTOP1: now also U2.27 (GPA6); no longer U2.28 (GPA7)
- net ENDSTOP2: now also U2.25 (GPA4); no longer U2.22 (GPA1)
- net GND: now also J14.2 (Pin_2), J15.2 (Pin_2)
- net M2_DIR: now reaches U2.8 (GPB7)
- net M2_DIR: now also A2.16 (DIR)
- net M_DIR renamed M1_DIR
- net M1_DIR: no longer A2.16 (DIR)
- new net: J16.1 (Pin_1), U2.28 (GPA7)
- new net: J16.2 (Pin_2), U2.23 (GPA2)
- new net: J16.3 (Pin_3), U2.22 (GPA1)
- new net: J16.4 (Pin_4), U2.21 (GPA0)
Other:
- note removed: "TODO: 4 endstop optice\n1 buton debounced click reconnect click and hold - apn la 90 de grade pe marginea pcb-ului sau undeva pe margine\n2 senzori pt a avea si presiunea atmosferica\n(ai o rezistenta prin care selectezi adresa)\nverifica gaurile de la cooler\nmicsoreaza placa, micsorand distanta dintr endstopuri\nvezi ce stie ciobu de-l avem pe spi si daca paote fi folosit ala pt a mana steppere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"
Changed lines of the file:
@@
 	2650 4050 2750 4050
 Text GLabel 750  3750 0    39   Input ~ 0
-M_DIR
+M1_DIR
 Text GLabel 750  3650 0    39   Input ~ 0
 M_STEP
@@
 	2750 3250 2750 3350
 Text GLabel 2750 3750 0    39   Input ~ 0
-M_DIR
+M2_DIR
 Text GLabel 2750 3650 0    39   Input ~ 0
 M_STEP
@@
 M_STEP
 Text GLabel 3050 5675 2    39   Input ~ 0
-M_DIR
+M1_DIR
 Text GLabel 3050 6175 2    39   Input ~ 0
 M2_EN
@@
 	1    0    0    -1
 $EndComp
-Text Notes 2150 -175 0    157  ~ 0
-TODO: 4 endstop optice\n1 buton debounced click reconnect click and hold - apn la 90 de grade pe marginea pcb-ului sau undeva pe margine\n2 senzori pt a avea si presiunea atmosferica\n(ai o rezistenta prin care selectezi adresa)\nverifica gaurile de la cooler\nmicsoreaza placa, micsorand distanta dintr endstopuri\nvezi ce stie ciobu de-l avem pe spi si daca paote fi folosit ala pt a mana steppere sau alte bazaconii (MCP23S17-E/SO)\nscoate endstopurile de pe placa, dar pastreaza rezistentele ca se muta doar bariera optica\nsenzorul de presiune pe placa - grija unde-l pui sa nu bata vntilatorul pe el\n\n\n4ms intre pulsurile de step - vezi daca mere cu mcp-u ala\n\n3 coolere\n1 buton de panica intre endstopuri \n\nSILK:\nlogo Symme3D,\nVentilaTM Mk1\nPCB Rev.XXX\ndata\n\n\n\n\n
 $Comp
 L power:+3V3 #PWR0122
@@
 Text GLabel 3050 5775 2    39   Input ~ 0
 BTN1
-Text GLabel 3050 6675 2    39   Input ~ 0
+Text GLabel 3050 6975 2    39   Input ~ 0
 BTN2
-Text GLabel 3050 6575 2    39   Input ~ 0
+Text GLabel 3050 6875 2    39   Input ~ 0
 ENDSTOP2
-Text GLabel 3050 7175 2    39   Input ~ 0
+Text GLabel 3050 7075 2    39   Input ~ 0
 ENDSTOP1
 Text GLabel 5825 2750 2    39   Input ~ 0
@@
 Text GLabel 8100 4200 2    39   Input ~ 0
 MISO
-Text GLabel 3050 6475 2    39   Input ~ 0
+Text GLabel 3050 6775 2    39   Input ~ 0
 CS1
 Text GLabel 8100 4000 2    39   Input ~ 0
@@
 Wire Wire Line
 	8500 3900 8100 3900
+Text GLabel 3050 6275 2    39   Input ~ 0
+M2_DIR
+$Comp
+L Connector:Conn_01x02_Male J14
+U 1 1 5E7D0D08
+P 1550 1750
+F 0 "J14" H 1658 1931 50  0000 C CNN
+F 1 "3v3spare" H 1658 1840 50  0000 C CNN
+F 2 "Connector_PinHeader_2.54mm:PinHeader_1x02_P2.54mm_Vertical" H 1550 1750 50  0001 C CNN
+F 3 "~" H 1550 1750 50  0001 C CNN
+	1    1550 1750
+	1    0    0    -1
+$EndComp
+$Comp
+L Connector:Conn_01x02_Male J15
+U 1 1 5E7D1F7D
+P 2275 1750
+F 0 "J15" H 2383 1931 50  0000 C CNN
+F 1 "3v3spare1" H 2383 1840 50  0000 C CNN
+F 2 "Connector_PinHeader_2.54mm:PinHeader_1x02_P2.54mm_Vertical" H 2275 1750 50  0001 C CNN
+F 3 "~" H 2275 1750 50  0001 C CNN
+	1    2275 1750
+	1    0    0    -1
+$EndComp
+$Comp
+L Connector:Conn_01x04_Male J16
+U 1 1 5E7D2D33
+P 3825 6675
+F 0 "J16" H 3750 6550 50  0000 C CNN
+F 1 "spare_pins" H 3625 6625 50  0000 C CNN
+F 2 "Connector_PinHeader_2.54mm:PinHeader_1x04_P2.54mm_Vertical" H 3825 6675 50  0001 C CNN
+F 3 "~" H 3825 6675 50  0001 C CNN
+	1    3825 6675
+	-1   0    0    1
+$EndComp
+Wire Wire Line
+	3050 6475 3625 6475
+Wire Wire Line
+	3050 6575 3625 6575
+Wire Wire Line
+	3050 6675 3625 6675
+Wire Wire Line
+	3050 7175 3625 7175
+Wire Wire Line
+	3625 7175 3625 6775
+$Comp
+L power:+3V3 #PWR0148
+U 1 1 5E8685DD
+P 2475 1750
+F 0 "#PWR0148" H 2475 1600 50  0001 C CNN
+F 1 "+3V3" V 2475 2000 50  0000 C CNN
+F 2 "" H 2475 1750 50  0001 C CNN
+F 3 "" H 2475 1750 50  0001 C CNN
+	1    2475 1750
+	0    1    1    0
+$EndComp
+$Comp
+L power:+3V3 #PWR0149
+U 1 1 5E86B723
+P 1750 1750
+F 0 "#PWR0149" H 1750 1600 50  0001 C CNN
+F 1 "+3V3" V 1750 2000 50  0000 C CNN
+F 2 "" H 1750 1750 50  0001 C CNN
+F 3 "" H 1750 1750 50  0001 C CNN
+	1    1750 1750
+	0    1    1    0
+$EndComp
+$Comp
+L power:GND #PWR0150
+U 1 1 5E86B9B1
+P 1750 1850
+F 0 "#PWR0150" H 1750 1600 50  0001 C CNN
+F 1 "GND" H 1755 1677 50  0000 C CNN
+F 2 "" H 1750 1850 50  0001 C CNN
+F 3 "" H 1750 1850 50  0001 C CNN
+	1    1750 1850
+	1    0    0    -1
+$EndComp
+$Comp
+L power:GND #PWR0151
+U 1 1 5E86BF64
+P 2475 1850
+F 0 "#PWR0151" H 2475 1600 50  0001 C CNN
+F 1 "GND" H 2480 1677 50  0000 C CNN
+F 2 "" H 2475 1850 50  0001 C CNN
+F 3 "" H 2475 1850 50  0001 C CNN
+	1    2475 1850
+	1    0    0    -1
+$EndComp
 $EndSCHEMATC
